File: Arduboy-clone.kicad_pcb (KiCad board)
At the start: 2 copper layers, 66.2 x 108.2 mm, 35 parts, among them J1 USB_C_Receptacle_USB2.0_16P, J2 Conn_01x08, SW1 SW_Push, SW2 SW_Push, SW3 SW_Push, SW4 SW_Push, SW5 SW_Push, SW6 SW_Push, SW7 SW_Push, U1 ATmega32U4-A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

Commit message: Generated Gerber File
Parts:
- moved R3 118.8 mm to (187.3, 138.6)
- moved R2 116.7 mm to (182.3, 138.7)
- moved C4 114.8 mm to (198.2, 98.5)
- moved C3 104.4 mm to (198.2, 93.1)
- moved Y1 102.3 mm to (198.2, 95.7)
- moved R1 90.3 mm to (167.0, 91.6), turned to 180 degrees
- moved R8 85.8 mm to (180.2, 84.1), turned to 180 degrees
- moved D2 80.7 mm to (173.8, 88.6), turned to 180 degrees
- moved U2 74.9 mm to (167.0, 89.0)
- moved R4 73.9 mm to (166.3, 93.3)
- moved L1 68.9 mm to (166.9, 85.0), turned to 180 degrees
- moved C2 52.7 mm to (171.1, 89.0), turned to -90 degrees
- moved D1 10.8 mm to (187.3, 128.5)
Routing:
- net Net-(BZ1--): track 0.00 -> 64.8 mm, vias 0 -> 2
- net Net-(BZ1-+): track 0.00 -> 47.2 mm, vias 0 -> 2
- net GND: track 0.00 -> 41.7 mm, vias 0 -> 4
- net Net-(D1-A): track 2.06 -> 19.4 mm, vias 0 -> 2
- net Net-(BT1-+): track 6.22 -> 23.5 mm
- net Net-(U1-XTAL1): track 0.00 -> 13.0 mm, vias 0 -> 2
- net Net-(U1-XTAL2): track 0.00 -> 11.2 mm, vias 0 -> 2
- net Net-(D2-A): track 0.00 -> 11.0 mm
- net 5V: track 123.0 -> 116.5 mm
- net Net-(U1-~{RESET}): track 54.2 -> 60.7 mm
- net Net-(J1-CC1): track 0.00 -> 4.08 mm
- net Net-(J1-CC2): track 0.00 -> 3.95 mm
- net Net-(U2-V_{FB}): track 0.00 -> 3.82 mm
- net Net-(U1-~{HWB}/PE2): track 0.00 -> 3.61 mm, vias 0 -> 2
- net Net-(U2-SW): track 0.00 -> 3.06 mm
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Other:
- board size 66.2 x 108.2 mm -> 65.1 x 106.8 mm

Commit message: Added Bom file and replaced display with a cheaper alternative
Parts:
- J2: value Conn_01x08 -> Conn_01x07; footprint Display:Adafruit_SSD1306 -> Connector_PinHeader_2.54mm:PinHeader_1x07_P2.54mm_Vertical
- moved R5 2.95 mm to (155.2, 47.2), turned to 90 degrees
- moved SW7 2.28 mm to (155.2, 50.0)
- moved J2 0.20 mm to (176.8, 46.1), turned to 90 degrees
Connections:
- J2 pad 2: unconnected-(J2-Pin_2-Pad2) -> 5V
- J2 pad 3: 5V -> /CLK
- J2 pad 4: /CS -> /MOSI
- J2 pad 7: /CLK -> /CS
Routing:
- net /CLK: track 64.1 -> 70.7 mm
- net /MOSI: track 63.2 -> 68.4 mm, vias 0 -> 2
- net /CS: track 42.0 -> 44.0 mm, vias 2 -> 1
- net 5V: track 116.5 -> 117.7 mm
- net /RES: track 40.9 -> 41.7 mm
- net /RESET: track 9.47 -> 8.87 mm
- net Net-(U1-~{RESET}): track 60.7 -> 61.3 mm
